Commit message: fast_livo

File: src/ranger_gazebo_experiments/urdf/ranger_mini_sim.urdf.xacro (robot description, xacro)
@@ -24,9 +24,11 @@
   <xacro:property name="wheel_x_offset" value="0.30"/>
   <xacro:property name="wheel_y_offset" value="0.35"/>
-  <xacro:property name="wheel_z_offset" value="-0.12"/>
+  <xacro:property name="wheel_z_offset" value="${wheel_radius}"/>
   <xacro:property name="lidar_x" value="0.30"/>
   <xacro:property name="lidar_y" value="0.0"/>
   <xacro:property name="lidar_z" value="0.70"/>
+  <xacro:property name="lidar_roll" value="0.0"/>
   <xacro:property name="lidar_pitch" value="0.523599"/>  <!-- 30 degrees -->
+  <xacro:property name="lidar_yaw" value="0.0"/>
   <xacro:property name="camera_x" value="0.35"/>
   <xacro:property name="camera_y" value="0.0"/>
@@ -79,5 +81,5 @@
     <link name="${prefix}_${name}_wheel_link">
       <visual>
-        <origin xyz="0 0 0" rpy="0 ${pi/2} 0"/>
+        <origin xyz="0 0 0" rpy="${pi/2} 0 0"/>
         <geometry>
           <cylinder radius="${wheel_radius}" length="${wheel_width}"/>
@@ -86,5 +88,5 @@
       </visual>
       <collision>
-        <origin xyz="0 0 0" rpy="0 ${pi/2} 0"/>
+        <origin xyz="0 0 0" rpy="${pi/2} 0 0"/>
         <geometry>
           <cylinder radius="${wheel_radius}" length="${wheel_width}"/>
@@ -126,5 +128,5 @@
     <parent link="base_link"/>
     <child link="livox_frame"/>
-    <origin xyz="${lidar_x} ${lidar_y} ${lidar_z}" rpy="0 ${lidar_pitch} 0"/>
+    <origin xyz="${lidar_x} ${lidar_y} ${lidar_z}" rpy="${lidar_roll} ${lidar_pitch} ${lidar_yaw}"/>
   </joint>
   <!-- ========== D435i Camera ========== -->
@@ -195,5 +197,5 @@
       <odometry_topic>odom</odometry_topic>
       <odometry_frame>odom</odometry_frame>
-      <robot_base_frame>base_link</robot_base_frame>
+      <robot_base_frame>base_footprint</robot_base_frame>
       <publish_odom_tf>true</publish_odom_tf>
       <publish_wheel_tf>false</publish_wheel_tf>
@@ -241,5 +243,5 @@
   </gazebo>
   <!-- D435i RGB Camera on color optical frame -->
-  <gazebo reference="camera_color_optical_frame">
+  <gazebo reference="camera_link">
     <sensor name="d435i_rgb" type="camera">
       <pose>0 0 0 0 0 0</pose>
@@ -271,5 +273,5 @@
   </gazebo>
   <!-- D435i Depth Camera — outputs depth image + pointcloud -->
-  <gazebo reference="camera_depth_optical_frame">
+  <gazebo reference="camera_link">
     <sensor name="d435i_depth" type="depth">
       <pose>0 0 0 0 0 0</pose>
